File: ESP32-CAM-USB-Flasher.kicad_pcb (KiCad board)
At the start: 2 copper layers, 27.9 x 30.5 mm, 10 parts, among them J1 LEFT, J2 USB_B_Micro, J3 RIGHT, Q1 UMH3N, Q2 AO3400A, U1 CH340C

Commit message: get the transistor footprint right
Parts:
- removed Q2: AO3400A, Package_TO_SOT_SMD:SOT-23_Handsoldering
- added C3: 10u, Capacitor_SMD:C_0805_2012Metric_Pad1.18x1.45mm_HandSolder, F.Cu at (62.7, 97.2)
- added C4: 100n, Capacitor_SMD:C_0805_2012Metric_Pad1.18x1.45mm_HandSolder, F.Cu at (66.7, 95.8)
- added C5: 22u, Capacitor_SMD:C_0805_2012Metric_Pad1.18x1.45mm_HandSolder, F.Cu at (62.2, 89.8)
- added Q3: S8050, Package_TO_SOT_SMD:SOT-23, F.Cu at (76.1, 91.3)
- added R2: 1M, Resistor_SMD:R_0805_2012Metric_Pad1.20x1.40mm_HandSolder, F.Cu at (76.1, 101.5)
- added R3: 10K, Resistor_SMD:R_0805_2012Metric_Pad1.20x1.40mm_HandSolder, F.Cu at (75.1, 86.7)
- added R4: 10K, Resistor_SMD:R_0805_2012Metric_Pad1.20x1.40mm_HandSolder, F.Cu at (77.1, 86.7)
- added R5: 470R, Resistor_SMD:R_0805_2012Metric_Pad1.20x1.40mm_HandSolder, F.Cu at (63.1, 80.1)
- added SW1: RESET, CPB:SW_Tact_C354947, F.Cu at (81.0, 100.3)
- added SW2: FLASH, CPB:SW_Tact_C354947, F.Cu at (58.4, 100.4)
- added U2: ME6217, Package_TO_SOT_SMD:SOT-23-5, F.Cu at (63.6, 93.8)
- Q1: value UMH3N -> S8050; footprint Package_TO_SOT_SMD:SOT-363_SC-70-6_Handsoldering -> Package_TO_SOT_SMD:SOT-23
- moved F1 6.56 mm to (66.9, 90.9)
- moved C1 5.57 mm to (64.0, 83.9)
- moved U1 5.51 mm to (69.1, 83.4)
- moved C2 5.51 mm to (69.3, 77.1)
- moved R1 2.18 mm to (76.2, 77.7), turned to 0 degrees
- moved Q1 2.17 mm to (76.1, 81.8)
Connections:
- J1 pad 1: Net-(J1-Pad1) -> GND
- J1 pad 4: (no net) -> unconnected-(J1-Pad4)
- J1 pad 5: Net-(J1-Pad1) -> GND
- J1 pad 7: (no net) -> unconnected-(J1-Pad7)
- J1 pad 8: (no net) -> +3V3
- J2 pad 4: (no net) -> unconnected-(J2-Pad4)
- J2 pad 6: GND -> Net-(J2-Pad6)
- J3 pad 1: (no net) -> unconnected-(J3-Pad1)
- J3 pad 2: (no net) -> unconnected-(J3-Pad2)
- J3 pad 3: (no net) -> unconnected-(J3-Pad3)
- J3 pad 4: (no net) -> unconnected-(J3-Pad4)
- J3 pad 5: (no net) -> unconnected-(J3-Pad5)
- J3 pad 6: (no net) -> unconnected-(J3-Pad6)
- J3 pad 7: Net-(J1-Pad1) -> GND
- J3 pad 8: +5V -> unconnected-(J3-Pad8)
- Q1 pad 1: /RTS -> Net-(Q1-Pad1)
- Q1 pad 2: /DTR -> /RTS
- Q1 pad 3: /GPIO0 -> /EN
- R1 pad 2: /RST -> /EN
- U1 pad 10: (no net) -> unconnected-(U1-Pad10)
- U1 pad 11: (no net) -> unconnected-(U1-Pad11)
- U1 pad 12: (no net) -> unconnected-(U1-Pad12)
- U1 pad 15: (no net) -> unconnected-(U1-Pad15)
- U1 pad 2: /URXD -> /CHTX
- U1 pad 7: (no net) -> unconnected-(U1-Pad7)
- U1 pad 8: (no net) -> unconnected-(U1-Pad8)
- U1 pad 9: (no net) -> unconnected-(U1-Pad9)
Routing:
- net Net-(J1-Pad1): track 48.5 -> 0.00 mm, vias 5 -> 0
- net /EN: track 0.00 -> 42.6 mm, vias 0 -> 2
- net Net-(J2-Pad6): track 0.00 -> 17.9 mm
- net /GPIO0: track 21.9 -> 32.0 mm, vias 1 -> 2
- net GND: track 12.4 -> 4.47 mm, vias 9 -> 20
- net +3V3: track 0.00 -> 7.90 mm, vias 0 -> 1
- net /URXD: track 10.8 -> 4.25 mm
- net +5V: track 50.3 -> 44.0 mm, vias 4 -> 3
- net /D-: track 9.10 -> 15.1 mm
- net /D+: track 10.8 -> 16.6 mm
- net /RST: track 5.60 -> 0.00 mm
- net /UTXD: track 14.5 -> 10.3 mm
- net Net-(Q1-Pad1): track 0.00 -> 3.05 mm
- net Net-(Q3-Pad1): track 0.00 -> 2.68 mm
- net /CHTX: track 0.00 -> 2.55 mm
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Other:
- outline, holes or cut-outs redrawn
- net class Default removed
